File: ksylen/ksylen.kicad_pcb (KiCad board)
At the start: 2 copper layers, 25 x 35 mm, 20 parts, among them J1 Conn2, J2 Conn1, U1 DIP-8, U2 LMC555, U3 DIP-16

Commit message: Add holes
Parts:
- added REF**: MountingHole_3.2mm_M3_Pad, MountingHole:MountingHole_3.2mm_M3_Pad, F.Cu at (94.0, 54.9)
- added REF**: MountingHole_3.2mm_M3_Pad, MountingHole:MountingHole_3.2mm_M3_Pad, F.Cu at (94.0, 80.9)
- added REF**: MountingHole_3.2mm_M3_Pad, MountingHole:MountingHole_3.2mm_M3_Pad, F.Cu at (121.0, 80.9)
- added REF**: MountingHole_3.2mm_M3_Pad, MountingHole:MountingHole_3.2mm_M3_Pad, F.Cu at (121.0, 54.9)
Routing:
- net V3V3: track 80.1 -> 0.00 mm, vias 2 -> 0
- net SCK: track 40.1 -> 0.00 mm
- net GND: track 35.0 -> 0.00 mm, vias 3 -> 0
- net MISO: track 27.5 -> 0.00 mm, vias 2 -> 0
- net CS: track 24.4 -> 0.00 mm
- net Net-(C4-Pad1): track 13.2 -> 0.00 mm
- net Net-(D1-Pad2): track 8.65 -> 0.00 mm, vias 1 -> 0
- net MOSI: track 6.66 -> 0.00 mm
- net Net-(R7-Pad1): track 5.34 -> 0.00 mm
- net Net-(C3-Pad2): track 4.99 -> 0.00 mm
Other:
- board size 25 x 35 mm -> 37 x 35 mm

Commit message: All components
Parts:
- added G***: LOGO, ksylen:xylene_pattern, F.Cu at (95.3, 67.7)
- added G***: LOGO, ksylen:xylene_pattern, F.Cu at (120.2, 67.7)
- moved C5 7.96 mm to (97.1, 61.5), turned to 270 degrees
- moved C6 4.63 mm to (94.3, 62.4)
- moved C2 3.80 mm to (107.8, 59.1)
- moved C1 1.51 mm to (107.8, 53.8), turned to 270 degrees
- moved C3 0.51 mm to (112.2, 64.6)
- moved R7 0.51 mm to (103.2, 64.6)
- moved C4 0.25 mm to (101.8, 73.5)
- moved J1 0.25 mm to (106.5, 76.0)
- moved J2 0.25 mm to (109.0, 76.0)
- moved R2 0.25 mm to (113.6, 81.1)
- moved R3 0.25 mm to (101.8, 81.1)
- moved R5 0.25 mm to (101.8, 76.0)
- moved R6 0.25 mm to (113.6, 76.0)
- moved R1 0.25 mm to (113.6, 78.5)
- moved R4 0.25 mm to (101.8, 78.5)
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
Commit message: Xylene
Parts:
- moved C4 11.8 mm to (113.6, 73.3), turned to 0 degrees
- moved D1 0.19 mm to (107.8, 83.9)
- turned R1 to 0 degrees
- turned R2 to 180 degrees
- turned R4 to 0 degrees
- turned R5 to 0 degrees
- turned R6 to 0 degrees
Routing:
- net V3V3: track 0.00 -> 84.9 mm, vias 0 -> 3
- net GND: track 0.00 -> 65.9 mm, vias 0 -> 3
- net MOSI: track 0.00 -> 59.2 mm, vias 0 -> 2
- net CS: track 0.00 -> 54.2 mm, vias 0 -> 2
- net SCK: track 0.00 -> 46.3 mm, vias 0 -> 2
- net MISO: track 0.00 -> 34.6 mm
- net Net-(D1-Pad2): track 0.00 -> 24.1 mm, vias 0 -> 1
- net Net-(C4-Pad1): track 0.00 -> 13.5 mm
- net Net-(R7-Pad1): track 0.00 -> 5.09 mm
- net Net-(J1-Pad1): track 0.00 -> 4.67 mm
- net Net-(J1-Pad3): track 0.00 -> 3.92 mm
- net Net-(J1-Pad2): track 0.00 -> 3.92 mm
- net Net-(J2-Pad3): track 0.00 -> 3.79 mm
- net Net-(C3-Pad2): track 0.00 -> 3.35 mm
